File: rt_board/hw/rt_board.sch (EAGLE design)
At the start: 60 parts, among them IC1 MCP170333MB, IC2/L1 TLE4935L, IC3/L2 TLE4935L, IC4/L1 TLE4935L, IC5/L2 TLE4935L, Q1 8MHz, U1 STM32F051R8T7, U2 SN74AVC4T245PW, U3 DRV8801PWP, U4 ACS712ELCTR-20A-T, U5 DRV8801PWP, U6 ACS712ELCTR-20A-T, X1 PWR, X2 LEFT, X3 RIGHT

Commit message: added LED to indicate circut is powered and one user-defined, controlled via uC
Parts:
- added LED1, LED2: GREEN, led:LEDCHIPLED_0603
- added R17: 470R, rcl:R-EU_R0603
- added U7: 2N7002BKW, 2n7002:2N7002BKW
Connections:
- new net N$43: LED1.A, R17.2
- new net N$44: U1.PB0, U7.GATE
- new net N$47: LED2.C, U7.DRAIN
- net +5V: now also LED2.A, R17.1
- net 0V: now also LED1.C, U7.SOURCE
- net N$17: now also U1.PA8; no longer U1.PA0
- net N$19: now also U1.PA9; no longer U1.PA1
Other:
- moved on the sheet: R4
Changed lines of the file:
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@@
 <part name="SUPPLY81" library="supply2" deviceset="0V" device=""/>
 <part name="SUPPLY82" library="supply2" deviceset="0V" device=""/>
+<part name="LED1" library="led" deviceset="LED" device="CHIPLED_0603" value="GREEN"/>
+<part name="R17" library="rcl" deviceset="R-EU_" device="R0603" value="470R"/>
+<part name="SUPPLY59" library="supply2" deviceset="+5V" device="" value="+3.3V"/>
+<part name="SUPPLY80" library="supply2" deviceset="0V" device=""/>
+<part name="U7" library="2n7002" deviceset="2N7002BKW" device=""/>
+<part name="SUPPLY83" library="supply2" deviceset="0V" device=""/>
+<part name="LED2" library="led" deviceset="LED" device="CHIPLED_0603" value="GREEN"/>
+<part name="SUPPLY84" library="supply2" deviceset="+5V" device="" value="+3.3V"/>
 </parts>
 <sheets>
@@
 <instance part="R3" gate="G$1" x="-48.26" y="-5.08" rot="R90"/>
 <instance part="SUPPLY35" gate="0V" x="-48.26" y="-12.7"/>
-<instance part="R4" gate="G$1" x="-50.8" y="15.24" rot="R90"/>
-<instance part="SUPPLY36" gate="+5V" x="-50.8" y="22.86"/>
+<instance part="R4" gate="G$1" x="-58.42" y="10.16" rot="R90"/>
+<instance part="SUPPLY36" gate="+5V" x="-58.42" y="20.32"/>
 <instance part="U2" gate="A" x="-172.72" y="66.04"/>
 <instance part="SV1" gate="1" x="-129.54" y="111.76" rot="R180"/>
@@
 <instance part="SUPPLY81" gate="0V" x="-177.8" y="-38.1"/>
 <instance part="SUPPLY82" gate="0V" x="-177.8" y="-195.58"/>
+<instance part="LED1" gate="G$1" x="-2.54" y="139.7"/>
+<instance part="R17" gate="G$1" x="-2.54" y="149.86" rot="R270"/>
+<instance part="SUPPLY59" gate="+5V" x="-2.54" y="160.02"/>
+<instance part="SUPPLY80" gate="0V" x="-2.54" y="129.54"/>
+<instance part="U7" gate="A" x="78.74" y="111.76"/>
+<instance part="SUPPLY83" gate="0V" x="73.66" y="109.22"/>
+<instance part="LED2" gate="G$1" x="114.3" y="124.46"/>
+<instance part="SUPPLY84" gate="+5V" x="114.3" y="132.08"/>
 </instances>
 <busses>
@@
 <wire x1="-177.8" y1="-193.04" x2="-180.34" y2="-193.04" width="0.1524" layer="91"/>
 </segment>
+<segment>
+<pinref part="LED1" gate="G$1" pin="C"/>
+<pinref part="SUPPLY80" gate="0V" pin="0V"/>
+<wire x1="-2.54" y1="132.08" x2="-2.54" y2="134.62" width="0.1524" layer="91"/>
+</segment>
+<segment>
+<pinref part="U7" gate="A" pin="SOURCE"/>
+<pinref part="SUPPLY83" gate="0V" pin="0V"/>
+<wire x1="73.66" y1="111.76" x2="78.74" y2="111.76" width="0.1524" layer="91"/>
+</segment>
 </net>
 <net name="+5V" class="0">
@@
 <pinref part="R4" gate="G$1" pin="2"/>
 <pinref part="SUPPLY36" gate="+5V" pin="+5V"/>
+<wire x1="-58.42" y1="15.24" x2="-58.42" y2="17.78" width="0.1524" layer="91"/>
 </segment>
 <segment>
@@
 <pinref part="SUPPLY27" gate="+5V" pin="+5V"/>
 <wire x1="-205.74" y1="73.66" x2="-190.5" y2="73.66" width="0.1524" layer="91"/>
+</segment>
+<segment>
+<pinref part="R17" gate="G$1" pin="1"/>
+<pinref part="SUPPLY59" gate="+5V" pin="+5V"/>
+<wire x1="-2.54" y1="157.48" x2="-2.54" y2="154.94" width="0.1524" layer="91"/>
+</segment>
+<segment>
+<pinref part="LED2" gate="G$1" pin="A"/>
+<pinref part="SUPPLY84" gate="+5V" pin="+5V"/>
+<wire x1="114.3" y1="129.54" x2="114.3" y2="127" width="0.1524" layer="91"/>
 </segment>
 </net>
@@
 <wire x1="-25.4" y1="10.16" x2="-50.8" y2="10.16" width="0.1524" layer="91"/>
 <wire x1="-50.8" y1="10.16" x2="-50.8" y2="5.08" width="0.1524" layer="91"/>
+<wire x1="-50.8" y1="5.08" x2="-58.42" y2="5.08" width="0.1524" layer="91"/>
 <pinref part="SWD" gate="1" pin="4"/>
-<wire x1="-50.8" y1="5.08" x2="-81.28" y2="5.08" width="0.1524" layer="91"/>
+<wire x1="-58.42" y1="5.08" x2="-81.28" y2="5.08" width="0.1524" layer="91"/>
 <pinref part="R4" gate="G$1" pin="1"/>
-<junction x="-50.8" y="10.16"/>
+<junction x="-58.42" y="5.08"/>
 </segment>
 </net>
@@
 <pinref part="R8" gate="G$1" pin="1"/>
 <wire x1="-185.42" y1="20.32" x2="-187.96" y2="20.32" width="0.1524" layer="91"/>
-<pinref part="U1" gate="A" pin="PA0"/>
 <wire x1="-187.96" y1="20.32" x2="-190.5" y2="20.32" width="0.1524" layer="91"/>
-<wire x1="-25.4" y1="48.26" x2="-139.7" y2="48.26" width="0.1524" layer="91"/>
-<wire x1="-139.7" y1="48.26" x2="-139.7" y2="30.48" width="0.1524" layer="91"/>
-<wire x1="-139.7" y1="30.48" x2="-187.96" y2="30.48" width="0.1524" layer="91"/>
-<wire x1="-187.96" y1="30.48" x2="-187.96" y2="20.32" width="0.1524" layer="91"/>
+<wire x1="-187.96" y1="27.94" x2="-187.96" y2="20.32" width="0.1524" layer="91"/>
 <junction x="-187.96" y="20.32"/>
+<pinref part="U1" gate="A" pin="PA8"/>
+<wire x1="-25.4" y1="27.94" x2="-187.96" y2="27.94" width="0.1524" layer="91"/>
 </segment>
 </net>
@@
 <pinref part="R10" gate="G$1" pin="1"/>
 <wire x1="-185.42" y1="0" x2="-187.96" y2="0" width="0.1524" layer="91"/>
-<pinref part="U1" gate="A" pin="PA1"/>
 <wire x1="-187.96" y1="0" x2="-190.5" y2="0" width="0.1524" layer="91"/>
-<wire x1="-25.4" y1="45.72" x2="-137.16" y2="45.72" width="0.1524" layer="91"/>
-<wire x1="-137.16" y1="45.72" x2="-137.16" y2="7.62" width="0.1524" layer="91"/>
-<wire x1="-137.16" y1="7.62" x2="-187.96" y2="7.62" width="0.1524" layer="91"/>
+<wire x1="-162.56" y1="25.4" x2="-162.56" y2="7.62" width="0.1524" layer="91"/>
+<wire x1="-162.56" y1="7.62" x2="-187.96" y2="7.62" width="0.1524" layer="91"/>
 <wire x1="-187.96" y1="7.62" x2="-187.96" y2="0" width="0.1524" layer="91"/>
 <junction x="-187.96" y="0"/>
+<pinref part="U1" gate="A" pin="PA9"/>
+<wire x1="-25.4" y1="25.4" x2="-162.56" y2="25.4" width="0.1524" layer="91"/>
 </segment>
 </net>
@@
 </segment>
 </net>
+<net name="N$43" class="0">
+<segment>
+<pinref part="LED1" gate="G$1" pin="A"/>
+<pinref part="R17" gate="G$1" pin="2"/>
+<wire x1="-2.54" y1="144.78" x2="-2.54" y2="142.24" width="0.1524" layer="91"/>
+</segment>
+</net>
+<net name="N$44" class="0">
+<segment>
+<pinref part="U1" gate="A" pin="PB0"/>
+<pinref part="U7" gate="A" pin="GATE"/>
+<wire x1="20.32" y1="86.36" x2="78.74" y2="86.36" width="0.1524" layer="91"/>
+<wire x1="78.74" y1="86.36" x2="78.74" y2="106.68" width="0.1524" layer="91"/>
+</segment>
+</net>
+<net name="N$47" class="0">
+<segment>
+<pinref part="U7" gate="A" pin="DRAIN"/>
+<pinref part="LED2" gate="G$1" pin="C"/>
+<wire x1="114.3" y1="119.38" x2="114.3" y2="111.76" width="0.1524" layer="91"/>
+</segment>
+</net>
